File: FPC_design/RigidPCBSensor_2withground17.brd (EAGLE design)
At the start: 34 x 46 mm, 34 parts

Commit message: comp vision work
Parts:
- removed E10, E11, E12, E13, E14, E15, E16, E9: TPSQTP15R, testpad:TP15R
- removed TP10, TP11, TP12, TP13, TP14, TP15, TP16, TP9: PTR1, RigidPCBSensor_1:TP10SQLONG
Connections:
- removed net N$10: E10.TP, TP10.TP
- removed net N$11: E11.TP, TP11.TP
- removed net N$12: E12.TP, TP12.TP
- removed net N$13: E13.TP, TP13.TP
- removed net N$14: E14.TP, TP14.TP
- removed net N$15: E15.TP, TP15.TP
- removed net N$16: E16.TP, TP16.TP
- removed net N$9: E9.TP, TP9.TP
Routing:
- net N$16: track 45.7 -> 0.00 mm, vias 1 -> 0
- net N$13: track 44.6 -> 0.00 mm, vias 3 -> 0
- net N$11: track 44.0 -> 0.00 mm, vias 1 -> 0
- net N$14: track 43.6 -> 0.00 mm, vias 1 -> 0
- net N$15: track 41.5 -> 0.00 mm, vias 1 -> 0
- net N$12: track 38.8 -> 0.00 mm, vias 1 -> 0
- net N$10: track 32.7 -> 0.00 mm, vias 1 -> 0
- net N$9: track 30.8 -> 0.00 mm, vias 3 -> 0
